File: BalBot/BalBot.kicad_pcb (KiCad board)
At the start: 2 copper layers, 76 parts, among them M1 Motor_N20, M2 Motor_N20, P1 FTSH-105-01-F-DV, P2 USB_OTG, P3 CONN_01X11, P4 CONN_01X11, P5 BATTERY, Q1 DTC114E, SW1 SW_RST, SW2 SW_USR1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

Commit message: Working On Layout
Parts:
- U9: footprint Housings_DFN_QFN:QFN-24_3x3mm_Pitch0.4mm_NoMask -> Housings_DFN_QFN:QFN-24_3x3mm_Pitch0.4mm
- moved D2 99.9 mm to (175.9, 35.1)
- moved JP1 99.9 mm to (169.2, 35.1)
- moved Q1 99.9 mm to (172.4, 32.0)
- moved R10 99.9 mm to (176.3, 37.6)
- moved C21 95.9 mm to (155.8, 108.8), turned to 90 degrees
- moved C28 91.2 mm to (155.2, 101.8)
- moved U9 87.7 mm to (155.0, 105.0)
- moved C22 83.4 mm to (154.2, 108.8), turned to 270 degrees
- moved U2 68.8 mm to (189.8, 89.9)
- moved C15 67.6 mm to (165.4, 74.6)
- moved P5 65.8 mm to (163.6, 50.2), turned to 270 degrees
- moved C24 65.1 mm to (159.1, 57.3), turned to 270 degrees
- moved C23 64.0 mm to (161.1, 57.3), turned to 270 degrees
- moved SW1 62.6 mm to (160.9, 70.5)
- moved M1 62.6 mm to (127.0, 130.0)
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Connections:
- net PD4/USB0_DM renamed USB0_D-
- net PD5/USB0_DP renamed USB0_D+
- net PWR_VBAT renamed PWR_VDD
- C13 pad 1: XOSC0 -> XOSC1
- C14 pad 2: XOSC1 -> XOSC0
- Y2 pad 1: XOSC1 -> XOSC0
- Y2 pad 2: XOSC0 -> XOSC1
Routing:
- net PWR_VDD: track 0.00 -> 92.9 mm
- net PWR_GND: track 0.00 -> 85.0 mm, vias 0 -> 20
- net RESET: track 0.00 -> 67.3 mm, vias 0 -> 2
- net +USB_VBUS: track 0.00 -> 55.3 mm, vias 0 -> 2
- net PB0/USB0_ID: track 0.00 -> 49.9 mm
- net USB0_D+: track 0.00 -> 49.8 mm
- net USB0_D-: track 0.00 -> 49.0 mm
- net PD6/QEI_PhA0: track 0.00 -> 45.0 mm
- net /DriveSystem/M1-: track 0.00 -> 29.4 mm
- net /DriveSystem/M2+: track 0.00 -> 29.1 mm
- net PB3/I2C_SDA: track 0.00 -> 27.1 mm, vias 0 -> 2
- net VIN: track 0.00 -> 26.8 mm
- net PB2/I2C_SCL: track 0.00 -> 25.8 mm, vias 0 -> 2
- net PC0/JTAG_TCK: track 0.00 -> 17.7 mm, vias 0 -> 2
- net PC3/JTAG_TDO: track 0.00 -> 17.4 mm
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- added copper zone on B.Cu, net Net-(C25-Pad1)
- added copper zone on F.Cu, net Net-(C25-Pad1)
- added copper zone on F.Cu, net PWR_GND
- added copper zone on F.Cu, net PWR_VDD
- added copper zone on F.Cu, net VIN
Other:
- board outline added: 80 x 100 mm
