File: BalBot/DriveSystem.sch (KiCad schematic (older format))
At the start: 17 parts, among them M1 Motor_N20, M2 Motor_N20, U4 TLE4946-2K, U5 TLE4946-2K, U6 DRV8848, U7 TLE4946-2K, U8 TLE4946-2K

Commit message: Started layout
Parts:
- C16, C19, C20: footprint (none) -> Capacitors_SMD:C_0402; DigiKey (none) -> 490-9997-1-ND
- C17: value 2.2uF 6.3V -> 2.2uF; footprint (none) -> Capacitors_SMD:C_0603; DigiKey (none) -> 490-12235-1-ND
- C18: footprint (none) -> Capacitors_SMD:C_0805; DigiKey (none) -> 490-12344-1-ND
- M1, M2: footprint (none) -> _BalBotLib:Motor_N20
- R11, R12, R13, R14, R15: footprint (none) -> Resistors_SMD:R_0805; DigiKey (none) -> 311-10.0KCRCT-ND
- U4, U5, U7, U8: footprint (none) -> TO_SOT_Packages_SMD:SC-59; DigiKey (none) -> TLE49462KHTSA1CT-ND
- U6: footprint (none) -> _BalBotLib:16-HTSSOP; DigiKey (none) -> 296-38514-5-ND
