File: BalBot/PowerSystem.sch (KiCad schematic (older format))
At the start: 12 parts, among them P5 BATTERY, SW4 SPST, U10 TPS562219DDF

Commit message: Started layout
Parts:
- added C29, C30: 22uF, Capacitors_SMD:C_0603, symbol C
- C23, C24: footprint (none) -> Capacitors_SMD:C_0805; DigiKey (none) -> 490-12344-1-ND
- C25: value C -> 0.1uF; footprint (none) -> Capacitors_SMD:C_0402; DigiKey (none) -> 490-9997-1-ND
- C26: value 8.2nF 1mOhm -> 8.2nF; footprint (none) -> Capacitors_SMD:C_0402; DigiKey (none) -> 490-6338-1-ND
- C27: value 22uF 3.71mOhm -> 22uF; footprint (none) -> Capacitors_SMD:C_0603; DigiKey (none) -> 1276-1193-1-ND
- D3: footprint (none) -> _BalBotLib:DO-214AC
- L1: footprint (none) -> _BalBotLib:IND_3.3uH_ASPI-0530LR-3R3M-T2; DigiKey (none) -> ASPI-0530LR-3R3M-T2CT-ND
- P5: footprint (none) -> _BalBotLib:XT60
- R16: footprint (none) -> Resistors_SMD:R_0805; DigiKey (none) -> 311-34.0KCRCT-ND
- R17: footprint (none) -> Resistors_SMD:R_0805; DigiKey (none) -> 311-10.0KCRCT-ND
- SW4: footprint (none) -> Pin_Headers:Pin_Header_Straight_1x02_Pitch2.54mm
- U10: footprint (none) -> TO_SOT_Packages_SMD:SOT-23-8; DigiKey (none) -> 296-48753-1-ND
Connections:
- net +3V3: now also C29.1, C30.1
- net GND: now also C29.2, C30.2
