File: BalBot/Sensors.sch (KiCad schematic (older format))
At the start: 3 parts, among them U9 MPU-6500

Commit message: Started layout
Parts:
- added C28: 0.1uF, Capacitors_SMD:C_0402, symbol C
- C21: footprint (none) -> Capacitors_SMD:C_0402; DigiKey (none) -> 490-9997-1-ND
- C22: value 2.2nF -> 10nF; footprint (none) -> Capacitors_SMD:C_0402; DigiKey (none) -> 490-16353-1-ND
- U9: footprint (none) -> Housings_DFN_QFN:QFN-24_3x3mm_Pitch0.4mm_NoMask; DigiKey (none) -> 1428-1011-1-ND
Connections:
- net +3V3: now also C28.1
- net GND: now also C28.2
Other:
- note added: "INERTIAL MEASUREMENT UNIT (MPU-6050)\nI2C ADDR: 1101000b"
- note removed: "I2C ADDR LSB Selection\nGND: 0, 3V3: 1"
- note removed: "INERTIAL MEASUREMENT UNIT (MPU-6050)\nI2C ADDR: 110100xb"
Changed lines of the file:
@@
 F 0 "U9" H 6200 3950 60  0000 C CNN
 F 1 "MPU-6500" H 6200 2850 60  0000 C CNN
-F 2 "" H 6200 3500 60  0001 C CNN
+F 2 "Housings_DFN_QFN:QFN-24_3x3mm_Pitch0.4mm_NoMask" H 6200 3500 60  0001 C CNN
 F 3 "" H 6200 3500 60  0001 C CNN
+F 4 "1428-1011-1-ND" H 6200 3400 60  0001 C CNN "DigiKey"
 	1    6200 3400
 	1    0    0    -1
 $EndComp
 $Comp
-L +3V3 #PWR45
+L +3V3 #PWR045
 U 1 1 5AEEBEFF
 P 5650 2950
-F 0 "#PWR45" H 5650 2800 50  0001 C CNN
+F 0 "#PWR045" H 5650 2800 50  0001 C CNN
 F 1 "+3V3" H 5650 3090 50  0000 C CNN
 F 2 "" H 5650 2950 50  0000 C CNN
@@
 	5650 3000 5700 3000
 $Comp
-L GND #PWR44
+L GND #PWR046
 U 1 1 5AEEBF28
 P 5150 3850
-F 0 "#PWR44" H 5150 3600 50  0001 C CNN
+F 0 "#PWR046" H 5150 3600 50  0001 C CNN
 F 1 "GND" H 5150 3700 50  0000 C CNN
 F 2 "" H 5150 3850 50  0000 C CNN
@@
 $EndComp
 Wire Wire Line
-	5150 3550 5150 3850
+	5150 3350 5150 3850
 Wire Wire Line
 	5150 3800 5700 3800
-Text GLabel 5650 3350 0    60   Input ~ 0
-ADO
-Wire Wire Line
-	5650 3350 5700 3350
-Text GLabel 8100 3400 1    60   Input ~ 0
-ADO
-$Comp
-L GND #PWR48
-U 1 1 5AEEBF6F
-P 8100 3450
-F 0 "#PWR48" H 8100 3200 50  0001 C CNN
-F 1 "GND" H 8100 3300 50  0000 C CNN
-F 2 "" H 8100 3450 50  0000 C CNN
-F 3 "" H 8100 3450 50  0000 C CNN
-	1    8100 3450
-	1    0    0    -1
-$EndComp
-Wire Wire Line
-	8100 3450 8100 3400
-Text Notes 7600 3050 0    60   ~ 0
-I2C ADDR LSB Selection\nGND: 0, 3V3: 1
+Wire Wire Line
+	5150 3350 5700 3350
 Text Notes 5000 2650 0    60   ~ 0
-INERTIAL MEASUREMENT UNIT (MPU-6050)\nI2C ADDR: 110100xb
+INERTIAL MEASUREMENT UNIT (MPU-6050)\nI2C ADDR: 1101000b
 Text HLabel 6750 3150 2    60   Input ~ 0
 I2C_SDA
@@
 F 0 "C21" H 9225 3450 50  0000 L CNN
 F 1 "0.1uF" H 9225 3250 50  0000 L CNN
-F 2 "" H 9238 3200 50  0000 C CNN
+F 2 "Capacitors_SMD:C_0402" H 9238 3200 50  0001 C CNN
 F 3 "" H 9200 3350 50  0000 C CNN
+F 4 "490-9997-1-ND" H 9200 3350 60  0001 C CNN "DigiKey"
 	1    9200 3350
 	1    0    0    -1
@@
 	9200 3150 9200 3200
 $Comp
-L GND #PWR49
+L GND #PWR048
 U 1 1 5AEEC123
 P 9200 3550
-F 0 "#PWR49" H 9200 3300 50  0001 C CNN
+F 0 "#PWR048" H 9200 3300 50  0001 C CNN
 F 1 "GND" H 9200 3400 50  0000 C CNN
 F 2 "" H 9200 3550 50  0000 C CNN
@@
 	9200 3550 9200 3500
 $Comp
-L GND #PWR46
+L GND #PWR049
 U 1 1 5AEEC189
 P 6750 3850
-F 0 "#PWR46" H 6750 3600 50  0001 C CNN
+F 0 "#PWR049" H 6750 3600 50  0001 C CNN
 F 1 "GND" H 6750 3700 50  0000 C CNN
 F 2 "" H 6750 3850 50  0000 C CNN
@@
 Text GLabel 9850 3150 0    60   Input ~ 0
 VDDIO
-$Comp
-L C C22
-U 1 1 5AEEC1CC
-P 9900 3350
-F 0 "C22" H 9925 3450 50  0000 L CNN
-F 1 "2.2nF" H 9925 3250 50  0000 L CNN
-F 2 "" H 9938 3200 50  0000 C CNN
-F 3 "" H 9900 3350 50  0000 C CNN
-	1    9900 3350
-	1    0    0    -1
-$EndComp
 Wire Wire Line
 	9850 3150 9900 3150
@@
 	9900 3150 9900 3200
 $Comp
-L GND #PWR50
+L GND #PWR050
 U 1 1 5AEEC205
 P 9900 3550
-F 0 "#PWR50" H 9900 3300 50  0001 C CNN
+F 0 "#PWR050" H 9900 3300 50  0001 C CNN
 F 1 "GND" H 9900 3400 50  0000 C CNN
 F 2 "" H 9900 3550 50  0000 C CNN
@@
 Connection ~ 5650 3250
 $Comp
-L +3V3 #PWR47
+L +3V3 #PWR051
 U 1 1 5AEEC37F
 P 7250 2950
-F 0 "#PWR47" H 7250 2800 50  0001 C CNN
+F 0 "#PWR051" H 7250 2800 50  0001 C CNN
 F 1 "+3V3" H 7250 3090 50  0000 C CNN
 F 2 "" H 7250 2950 50  0000 C CNN
@@
 Wire Wire Line
 	7250 3350 6700 3350
+$Comp
+L +3V3 #PWR052
+U 1 1 5AEFF15D
+P 10400 3150
+F 0 "#PWR052" H 10400 3000 50  0001 C CNN
+F 1 "+3V3" H 10400 3290 50  0000 C CNN
+F 2 "" H 10400 3150 50  0000 C CNN
+F 3 "" H 10400 3150 50  0000 C CNN
+	1    10400 3150
+	1    0    0    -1
+$EndComp
+$Comp
+L GND #PWR053
+U 1 1 5AEFF1B6
+P 10400 3550
+F 0 "#PWR053" H 10400 3300 50  0001 C CNN
+F 1 "GND" H 10400 3400 50  0000 C CNN
+F 2 "" H 10400 3550 50  0000 C CNN
+F 3 "" H 10400 3550 50  0000 C CNN
+	1    10400 3550
+	1    0    0    -1
+$EndComp
+$Comp
+L C C28
+U 1 1 5AEFF1CB
+P 10400 3350
+F 0 "C28" H 10425 3450 50  0000 L CNN
+F 1 "0.1uF" H 10425 3250 50  0000 L CNN
+F 2 "Capacitors_SMD:C_0402" H 10438 3200 50  0001 C CNN
+F 3 "" H 10400 3350 50  0000 C CNN
+F 4 "490-9997-1-ND" H 10400 3350 60  0001 C CNN "DigiKey"
+	1    10400 3350
+	1    0    0    -1
+$EndComp
+Wire Wire Line
+	10400 3150 10400 3200
+Wire Wire Line
+	10400 3500 10400 3550
+$Comp
+L C C22
+U 1 1 5AEFF3A1
+P 9900 3350
+F 0 "C22" H 9925 3450 50  0000 L CNN
+F 1 "10nF" H 9925 3250 50  0000 L CNN
+F 2 "Capacitors_SMD:C_0402" H 9938 3200 50  0001 C CNN
+F 3 "" H 9900 3350 50  0000 C CNN
+F 4 "490-16353-1-ND" H 9900 3350 60  0001 C CNN "DigiKey"
+	1    9900 3350
+	1    0    0    -1
+$EndComp
+Connection ~ 5150 3550
 $EndSCHEMATC

Commit message: Working On Layout
Parts:
- U9: footprint Housings_DFN_QFN:QFN-24_3x3mm_Pitch0.4mm_NoMask -> Housings_DFN_QFN:QFN-24_3x3mm_Pitch0.4mm
Changed lines of the file:
@@
 EESchema Schematic File Version 2
+LIBS:BalBot-rescue
 LIBS:power
 LIBS:device
@@
 F 0 "U9" H 6200 3950 60  0000 C CNN
 F 1 "MPU-6500" H 6200 2850 60  0000 C CNN
-F 2 "Housings_DFN_QFN:QFN-24_3x3mm_Pitch0.4mm_NoMask" H 6200 3500 60  0001 C CNN
+F 2 "Housings_DFN_QFN:QFN-24_3x3mm_Pitch0.4mm" H 6200 3500 60  0001 C CNN
 F 3 "" H 6200 3500 60  0001 C CNN
 F 4 "1428-1011-1-ND" H 6200 3400 60  0001 C CNN "DigiKey"
@@
 	9200 3150 9200 3200
 $Comp
-L GND #PWR048
+L GND #PWR047
 U 1 1 5AEEC123
 P 9200 3550
-F 0 "#PWR048" H 9200 3300 50  0001 C CNN
+F 0 "#PWR047" H 9200 3300 50  0001 C CNN
 F 1 "GND" H 9200 3400 50  0000 C CNN
 F 2 "" H 9200 3550 50  0000 C CNN
@@
 	9200 3550 9200 3500
 $Comp
-L GND #PWR049
+L GND #PWR048
 U 1 1 5AEEC189
 P 6750 3850
-F 0 "#PWR049" H 6750 3600 50  0001 C CNN
+F 0 "#PWR048" H 6750 3600 50  0001 C CNN
 F 1 "GND" H 6750 3700 50  0000 C CNN
 F 2 "" H 6750 3850 50  0000 C CNN
@@
 	9900 3150 9900 3200
 $Comp
-L GND #PWR050
+L GND #PWR049
 U 1 1 5AEEC205
 P 9900 3550
-F 0 "#PWR050" H 9900 3300 50  0001 C CNN
+F 0 "#PWR049" H 9900 3300 50  0001 C CNN
 F 1 "GND" H 9900 3400 50  0000 C CNN
 F 2 "" H 9900 3550 50  0000 C CNN
@@
 Connection ~ 5650 3250
 $Comp
-L +3V3 #PWR051
+L +3V3 #PWR050
 U 1 1 5AEEC37F
 P 7250 2950
-F 0 "#PWR051" H 7250 2800 50  0001 C CNN
+F 0 "#PWR050" H 7250 2800 50  0001 C CNN
 F 1 "+3V3" H 7250 3090 50  0000 C CNN
 F 2 "" H 7250 2950 50  0000 C CNN
@@
 	7250 3350 6700 3350
 $Comp
-L +3V3 #PWR052
+L +3V3 #PWR051
 U 1 1 5AEFF15D
 P 10400 3150
-F 0 "#PWR052" H 10400 3000 50  0001 C CNN
+F 0 "#PWR051" H 10400 3000 50  0001 C CNN
 F 1 "+3V3" H 10400 3290 50  0000 C CNN
 F 2 "" H 10400 3150 50  0000 C CNN
@@
 $EndComp
 $Comp
-L GND #PWR053
+L GND #PWR052
 U 1 1 5AEFF1B6
 P 10400 3550
-F 0 "#PWR053" H 10400 3300 50  0001 C CNN
+F 0 "#PWR052" H 10400 3300 50  0001 C CNN
 F 1 "GND" H 10400 3400 50  0000 C CNN
 F 2 "" H 10400 3550 50  0000 C CNN
